File: openmv4_cam_direct_mount/basev2.kicad_pcb (KiCad board)
At the start: 4 copper layers, 36 x 34 mm, 62 parts, among them Q1 BSS138, Q2 Si2301BDS, U1 STM32H743VIT6, U5 TPS731XX, U8 PAM2305AABADJ, X1 MF-CON-MICROUSB-RIGHT, X2 USD-1040310811, Y1 7S-12.000MAHE-T

Commit message: Changes to KiCAD
Parts:
- moved X1 47.6 mm to (109.8, 123.0), turned to 315 degrees
- moved D3 47.5 mm to (103.9, 119.7), turned to 135 degrees
- moved L3 46.5 mm to (100.5, 115.9), turned to 225 degrees
- moved R9 46.4 mm to (102.5, 117.3), turned to 225 degrees
- moved R10 45.3 mm to (99.6, 113.4), turned to 225 degrees
- moved C2 45.2 mm to (98.3, 112.4), turned to 225 degrees
- moved Q2 45.2 mm to (106.0, 117.6), turned to 315 degrees
- moved L2 44.1 mm to (109.8, 117.9), turned to 135 degrees
- moved U8 44.0 mm to (102.8, 113.6), turned to 135 degrees
- moved C8 43.8 mm to (112.4, 118.7), turned to 225 degrees
- moved C44 43.7 mm to (105.1, 114.7), turned to 45 degrees
- moved C49 43.4 mm to (107.6, 115.7), turned to 135 degrees
- moved R5 42.9 mm to (101.8, 111.2), turned to 225 degrees
- moved C4 38.8 mm to (102.1, 104.6), turned to 225 degrees
- moved C5 38.8 mm to (100.9, 103.5), turned to 225 degrees
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Routing:
- net VBUS: track 18.8 -> 0.00 mm, vias 2 -> 0
- net /SDIO_CMD: track 22.1 -> 9.58 mm
- net /SDIO_CLK: track 16.4 -> 4.07 mm
- net /TIM4_CH1: track 14.9 -> 4.59 mm, vias 1 -> 0
- net /SWDIO: track 9.37 -> 0.00 mm
- net /SWCLK: track 13.2 -> 4.20 mm, vias 1 -> 0
- net /SPI3_SCLK/TRACESWO: track 12.5 -> 3.77 mm, vias 1 -> 0
- net /SDIO_D3: track 18.3 -> 10.2 mm
- net /TIM4_CH3: track 14.2 -> 6.35 mm, vias 2 -> 1
- net /TIM4_CH2: track 14.0 -> 6.37 mm, vias 1 -> 0
- net /BOOT0: track 26.9 -> 19.7 mm
- net /SDIO_D2: track 17.4 -> 10.8 mm
- net /NRST: track 26.7 -> 20.7 mm
- net /SD_CD: track 15.6 -> 10.3 mm, vias 2 -> 1
- net /DCMI_D0: track 4.23 -> 0.57 mm, vias 2 -> 1
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