File: openmv4_cam_direct_mount/base.sch (KiCad schematic (older format))
At the start: 57 parts, among them J5 XF2M-1015-1A, Q1 BSS138, Q2 Si2301BDS, U1 STM32H743VIT6, U2 OV7725, U5 TPS731XX, U8 PAM2305AABADJ, X1 MF-CON-MICROUSB-RIGHT, X2 USD-1040310811, Y1 7S-12.000MAHE-T

Commit message: fab cleanup finished
Parts:
- added R6, R7: 0, base:0603-RES, symbol base-eagle-import:RESISTOR0603-RES
- J5: symbol XF2M-1015-1A:XF2M-1015-1A -> base-rescue:XF2M-1015-1A-XF2M-1015-1A
- U2: symbol openmv3-eagle-import:OV7725 -> base-rescue:OV7725-openmv3-eagle-import
Connections:
- net labels removed: BATT_N
Changed lines of the file:
@@
 	11100 3500 11100 4700
 $Comp
-L openmv3-eagle-import:OV7725 U2
+L base-rescue:OV7725-openmv3-eagle-import U2
 U 1 1 5DA85E18
 P 14550 9150
@@
 	9000 8100 9800 8100
 $Comp
-L XF2M-1015-1A:XF2M-1015-1A J5
+L base-rescue:XF2M-1015-1A-XF2M-1015-1A J5
 U 1 1 5DBF5F14
 P 12750 1850
@@
 $EndComp
 Wire Wire Line
-	13650 1950 13850 1950
-Wire Wire Line
 	13650 2050 13850 2050
 Wire Wire Line
 	13650 2150 13850 2150
 Wire Wire Line
-	13650 2250 13850 2250
-Wire Wire Line
 	12750 2250 12500 2250
 Wire Wire Line
@@
 Wire Wire Line
 	12750 2050 12500 2050
-Wire Wire Line
-	12750 1950 12500 1950
-Wire Wire Line
-	12750 1850 12500 1850
-Text Label 12750 2050 2    50   ~ 0
+Text Label 13850 2050 0    50   ~ 0
 PWR_EN
+Text Label 12500 2050 2    50   ~ 0
+SPI2_MOSI
+Text Label 12500 2250 2    50   ~ 0
+SPI2_NSS
+Text Label 12500 2150 2    50   ~ 0
+SPI2_MISO
 Text Label 13850 2150 0    50   ~ 0
-SPI2_MOSI
-Text Label 13850 2050 0    50   ~ 0
-SPI2_NSS
-Text Label 12400 2150 0    50   ~ 0
-SPI2_MISO
-Text Label 12400 2250 0    50   ~ 0
 SPI2_SCLK
-Text Label 13850 1950 0    50   ~ 0
-BATT_N
 $Comp
 L base-eagle-import:VCC #P+0102
 U 1 1 5DB9CD98
-P 12500 1500
-F 0 "#P+0102" H 12500 1500 50  0001 C CNN
-F 1 "VCC" V 12400 1400 59  0000 L BNN
-F 2 "" H 12500 1500 50  0001 C CNN
-F 3 "" H 12500 1500 50  0001 C CNN
-	1    12500 1500
-	1    0    0    -1
-$EndComp
-Wire Wire Line
-	12500 1850 12500 1600
+P 12600 1450
+F 0 "#P+0102" H 12600 1450 50  0001 C CNN
+F 1 "VCC" V 12500 1350 59  0000 L BNN
+F 2 "" H 12600 1450 50  0001 C CNN
+F 3 "" H 12600 1450 50  0001 C CNN
+	1    12600 1450
+	1    0    0    -1
+$EndComp
 $Comp
 L base-eagle-import:GND #GND013
@@
 	0    1    1    0
 $EndComp
+Wire Wire Line
+	13650 1950 13650 1850
+Connection ~ 13650 1850
+$Comp
+L base-eagle-import:RAW #RAW0101
+U 1 1 5DC00135
+P 11800 1550
+F 0 "#RAW0101" H 11800 1550 50  0001 C CNN
+F 1 "RAW" V 11700 1450 59  0000 L BNN
+F 2 "" H 11800 1550 50  0001 C CNN
+F 3 "" H 11800 1550 50  0001 C CNN
+	1    11800 1550
+	1    0    0    -1
+$EndComp
+$Comp
+L base-eagle-import:RESISTOR0603-RES R6
+U 1 1 5DC01702
+P 12000 1700
+F 0 "R6" H 11950 1559 59  0000 L BNN
+F 1 "0" H 11950 1770 59  0000 L BNN
+F 2 "base:0603-RES" H 12000 1700 50  0001 C CNN
+F 3 "" H 12000 1700 50  0001 C CNN
+	1    12000 1700
+	-1   0    0    1
+$EndComp
+$Comp
+L base-eagle-import:RESISTOR0603-RES R7
+U 1 1 5DC02332
+P 12400 1700
+F 0 "R7" H 12350 1559 59  0000 L BNN
+F 1 "0" H 12350 1770 59  0000 L BNN
+F 2 "base:0603-RES" H 12400 1700 50  0001 C CNN
+F 3 "" H 12400 1700 50  0001 C CNN
+	1    12400 1700
+	-1   0    0    1
+$EndComp
+Wire Wire Line
+	12200 1700 12200 1850
+Wire Wire Line
+	12200 1850 12750 1850
+Connection ~ 12200 1700
+Wire Wire Line
+	12600 1550 12600 1700
+Wire Wire Line
+	11800 1550 11800 1700
 $EndSCHEMATC
