File: !OpenMV_Master_Design/openmv4_cam_direct_mount/base.kicad_pcb (KiCad board)
At the start: 4 copper layers, 36 x 34 mm, 58 parts, among them J5 XF2M-1015-1A, Q1 BSS138, Q2 Si2301BDS, U1 STM32H743VIT6, U2 OV7725, U5 TPS731XX, U8 PAM2305AABADJ, X1 MF-CON-MICROUSB-RIGHT, X2 USD-1040310811, Y1 7S-12.000MAHE-T

Commit message: Folder Tidy
Other:
- board size 36 x 34 mm -> 75.2 x 45.2 mm
Changed lines of the file:
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@@
   (general
     (thickness 1.6)
-    (drawings 80)
+    (drawings 96)
     (tracks 775)
     (zones 0)
@@
       (net 97 /LED_IR) (solder_mask_margin 0.0762))
     (model "C:/Program Files/KiCad/share/kicad/modules/Package_QFP.pretty/LQFP-100_14x14mm_P0.5mm.kicad_mod"
-      (at (xyz 0 0 0))
+      (offset (xyz 10 0 0))
       (scale (xyz 1 1 1))
-      (rotate (xyz 0 0 0))
+      (rotate (xyz 0 0 90))
+    )
+    (model C:/Users/nickg/Desktop/AA236/OpenMV_Camera/OpenMV_Camera-max-fab-review1/Custom_CAD_Components/LQFP100.STEP
+      (offset (xyz -7 -7 0))
+      (scale (xyz 1 1 1))
+      (rotate (xyz -90 0 0))
     )
   )
@@
       (net 43 /SPI3_SCLK/TRACESWO) (solder_mask_margin 0.0762))
   )
+  (gr_line (start 196.199999 113.399999) (end 179.199999 113.399999) (layer Edge.Cuts) (width 0.2))
+  (gr_line (start 179.199999 96.4) (end 196.199999 96.4) (layer Edge.Cuts) (width 0.2))
+  (gr_line (start 171.3 130.2) (end 169.699999 130.199999) (layer Edge.Cuts) (width 0.2))
+  (gr_line (start 169.699999 130.199999) (end 169.699999 88.2) (layer Edge.Cuts) (width 0.2))
+  (gr_line (start 179.199999 113.399999) (end 179.199999 96.4) (layer Edge.Cuts) (width 0.2))
+  (gr_line (start 171.3 131.8) (end 171.3 130.2) (layer Edge.Cuts) (width 0.2))
+  (gr_line (start 196.199999 96.4) (end 196.199999 113.399999) (layer Edge.Cuts) (width 0.2))
+  (gr_line (start 169.699999 88.2) (end 171.3 88.2) (layer Edge.Cuts) (width 0.2))
+  (gr_line (start 204.099998 130.199999) (end 204.099998 131.8) (layer Edge.Cuts) (width 0.2))
+  (gr_line (start 205.699999 88.2) (end 205.699998 130.199999) (layer Edge.Cuts) (width 0.2))
+  (gr_line (start 205.699998 130.199999) (end 204.099998 130.199999) (layer Edge.Cuts) (width 0.2))
+  (gr_line (start 171.3 86.6) (end 204.099998 86.6) (layer Edge.Cuts) (width 0.2))
+  (gr_line (start 204.099998 131.8) (end 171.3 131.8) (layer Edge.Cuts) (width 0.2))
+  (gr_line (start 204.099998 88.2) (end 205.699999 88.2) (layer Edge.Cuts) (width 0.2))
+  (gr_line (start 204.099998 86.6) (end 204.099998 88.2) (layer Edge.Cuts) (width 0.2))
+  (gr_line (start 171.3 88.2) (end 171.3 86.6) (layer Edge.Cuts) (width 0.2))
   (gr_text v00 (at 165.80612 112.8776 90) (layer F.SilkS)
     (effects (font (size 0.77216 0.77216) (thickness 0.16256)) (justify left bottom))

Commit message: Catching remote up
Other:
- board size 75.2 x 45.2 mm -> 88.3 x 46.8 mm
Changed lines of the file:
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@@
     (pad 1 smd rect (at -0.85 0 270) (size 1.1 1) (layers Top F.Paste F.Mask)
       (net 3 VCC) (solder_mask_margin 0.0762))
+    (model ${KISYS3DMOD}/Resistor_SMD.3dshapes/R_0603_1608Metric.step
+      (at (xyz 0 0 0))
+      (scale (xyz 1 1 1))
+      (rotate (xyz 0 0 0))
+    )
   )
   (module base:0603-RES (layer Top)
@@
     (pad 1 smd rect (at -0.85 0 270) (size 1.1 1) (layers Top F.Paste F.Mask)
       (net 117 "Net-(J5-Pad1)") (solder_mask_margin 0.0762))
+    (model ${KISYS3DMOD}/Resistor_SMD.3dshapes/R_0603_1608Metric.step
+      (at (xyz 0 0 0))
+      (scale (xyz 1 1 1))
+      (rotate (xyz 0 0 0))
+    )
   )
   (module XF2M-1015-1A:XF2M-1015-1A (layer Bottom)
@@
       (rotate (xyz 0 0 90))
     )
-    (model C:/Users/nickg/Desktop/AA236/OpenMV_Camera/OpenMV_Camera-max-fab-review1/Custom_CAD_Components/LQFP100.STEP
+    (model C:/Users/nickg/Desktop/AA236/OpenMV_Camera/!OpenMV_Master_Design/Custom_CAD_Components/LQFP100.STEP
       (offset (xyz -7 -7 0))
       (scale (xyz 1 1 1))
@@
       (net 43 /SPI3_SCLK/TRACESWO) (solder_mask_margin 0.0762))
   )
-  (gr_line (start 196.199999 113.399999) (end 179.199999 113.399999) (layer Edge.Cuts) (width 0.2))
-  (gr_line (start 179.199999 96.4) (end 196.199999 96.4) (layer Edge.Cuts) (width 0.2))
-  (gr_line (start 171.3 130.2) (end 169.699999 130.199999) (layer Edge.Cuts) (width 0.2))
-  (gr_line (start 169.699999 130.199999) (end 169.699999 88.2) (layer Edge.Cuts) (width 0.2))
-  (gr_line (start 179.199999 113.399999) (end 179.199999 96.4) (layer Edge.Cuts) (width 0.2))
-  (gr_line (start 171.3 131.8) (end 171.3 130.2) (layer Edge.Cuts) (width 0.2))
-  (gr_line (start 196.199999 96.4) (end 196.199999 113.399999) (layer Edge.Cuts) (width 0.2))
-  (gr_line (start 169.699999 88.2) (end 171.3 88.2) (layer Edge.Cuts) (width 0.2))
-  (gr_line (start 204.099998 130.199999) (end 204.099998 131.8) (layer Edge.Cuts) (width 0.2))
-  (gr_line (start 205.699999 88.2) (end 205.699998 130.199999) (layer Edge.Cuts) (width 0.2))
-  (gr_line (start 205.699998 130.199999) (end 204.099998 130.199999) (layer Edge.Cuts) (width 0.2))
-  (gr_line (start 171.3 86.6) (end 204.099998 86.6) (layer Edge.Cuts) (width 0.2))
-  (gr_line (start 204.099998 131.8) (end 171.3 131.8) (layer Edge.Cuts) (width 0.2))
-  (gr_line (start 204.099998 88.2) (end 205.699999 88.2) (layer Edge.Cuts) (width 0.2))
-  (gr_line (start 204.099998 86.6) (end 204.099998 88.2) (layer Edge.Cuts) (width 0.2))
-  (gr_line (start 171.3 88.2) (end 171.3 86.6) (layer Edge.Cuts) (width 0.2))
+  (gr_line (start 192.300001 99.050001) (end 209.300001 99.050001) (layer Edge.Cuts) (width 0.2))
+  (gr_line (start 209.300001 116.05) (end 192.300001 116.05) (layer Edge.Cuts) (width 0.2))
+  (gr_line (start 217.2 82.25) (end 218.800001 82.250001) (layer Edge.Cuts) (width 0.2))
+  (gr_line (start 218.800001 82.250001) (end 218.800001 124.25) (layer Edge.Cuts) (width 0.2))
+  (gr_line (start 209.300001 99.050001) (end 209.300001 116.05) (layer Edge.Cuts) (width 0.2))
+  (gr_line (start 217.2 80.65) (end 217.2 82.25) (layer Edge.Cuts) (width 0.2))
+  (gr_line (start 192.300001 116.05) (end 192.300001 99.050001) (layer Edge.Cuts) (width 0.2))
+  (gr_line (start 218.800001 124.25) (end 217.2 124.25) (layer Edge.Cuts) (width 0.2))
+  (gr_line (start 184.400002 82.250001) (end 184.400002 80.65) (layer Edge.Cuts) (width 0.2))
+  (gr_line (start 182.800001 124.25) (end 182.800002 82.250001) (layer Edge.Cuts) (width 0.2))
+  (gr_line (start 182.800002 82.250001) (end 184.400002 82.250001) (layer Edge.Cuts) (width 0.2))
+  (gr_line (start 217.2 125.85) (end 184.400002 125.85) (layer Edge.Cuts) (width 0.2))
+  (gr_line (start 184.400002 80.65) (end 217.2 80.65) (layer Edge.Cuts) (width 0.2))
+  (gr_line (start 184.400002 124.25) (end 182.800001 124.25) (layer Edge.Cuts) (width 0.2))
+  (gr_line (start 184.400002 125.85) (end 184.400002 124.25) (layer Edge.Cuts) (width 0.2))
+  (gr_line (start 217.2 124.25) (end 217.2 125.85) (layer Edge.Cuts) (width 0.2))
   (gr_text v00 (at 165.80612 112.8776 90) (layer F.SilkS)
     (effects (font (size 0.77216 0.77216) (thickness 0.16256)) (justify left bottom))
