File: !OpenMV_Master_Design/openmv4_cam_v3/base.sch (KiCad schematic (older format))
At the start: 59 parts, among them J5 XF2M-1015-1A, Q1 BSS138, Q2 Si2301BDS, U1 STM32H743VIT6, U2 OV7725, U5 TPS731XX, U8 PAM2305AABADJ, X1 MF-CON-MICROUSB-RIGHT, X2 USD-1040310811, Y1 7S-12.000MAHE-T

Commit message: Starting V3 (using MV4 style connector)
Parts:
- J5: footprint XF2M-1015-1A -> base:XF2M-1015-1A
- gave numbers to parts that had none: 2
Changed lines of the file:
@@
 F 0 "J5" H 13200 2115 50  0000 C CNN
 F 1 "XF2M-1015-1A" H 13200 2024 50  0000 C CNN
-F 2 "XF2M-1015-1A" H 13500 1950 50  0001 L CNN
+F 2 "base:XF2M-1015-1A" H 13500 1950 50  0001 L CNN
 F 3 "https://componentsearchengine.com/Datasheets/3/XF2M-1015-1A.pdf" H 13500 1850 50  0001 L CNN
 F 4 "0.5mm Rotary backlock 10 way Omron XF2M Series 0.5mm Pitch 10 Way Right Angle SMT Female FPC Connector Locking Mechanism, Top and Bottom Contact" H 13500 1750 50  0001 L CNN "Description"
@@
 Connection ~ 13650 1850
 $Comp
-L base-eagle-import:RAW #RAW?
+L base-eagle-import:RAW #RAW0101
 U 1 1 5DC00135
 P 11800 1550
-F 0 "#RAW?" H 11800 1550 50  0001 C CNN
+F 0 "#RAW0101" H 11800 1550 50  0001 C CNN
 F 1 "RAW" V 11700 1450 59  0000 L BNN
 F 2 "" H 11800 1550 50  0001 C CNN
@@
 $EndComp
 $Comp
-L base-eagle-import:RESISTOR0603-RES R?
+L base-eagle-import:RESISTOR0603-RES R6
 U 1 1 5DC01702
 P 12000 1700
-F 0 "R?" H 11950 1559 59  0000 L BNN
+F 0 "R6" H 11950 1559 59  0000 L BNN
 F 1 "0" H 11950 1770 59  0000 L BNN
 F 2 "base:0603-RES" H 12000 1700 50  0001 C CNN
@@
 $EndComp
 $Comp
-L base-eagle-import:RESISTOR0603-RES R?
+L base-eagle-import:RESISTOR0603-RES R7
 U 1 1 5DC02332
 P 12400 1700
-F 0 "R?" H 12350 1559 59  0000 L BNN
+F 0 "R7" H 12350 1559 59  0000 L BNN
 F 1 "0" H 12350 1770 59  0000 L BNN
 F 2 "base:0603-RES" H 12400 1700 50  0001 C CNN
