File: !OpenMV_Master_Design/openmv4_cam_v2/base.sch (KiCad schematic (older format))
At the start: 59 parts, among them J5 XF2M-1015-1A, Q1 BSS138, Q2 Si2301BDS, U1 STM32H743VIT6, U2 OV7725, U5 TPS731XX, U8 PAM2305AABADJ, X1 MF-CON-MICROUSB-RIGHT, X2 USD-1040310811, Y1 7S-12.000MAHE-T

Commit message: Moved the flat flex connector to suit main board design
Parts:
- removed C12: 47uF, openmv3:EIA3216, symbol base-eagle-import:CAP_POL1206
- removed C15, C16, C17, C19: 0.1uF, openmv3:0603-CAP, symbol base-eagle-import:CAP0603-CAP
- removed C18: 4.7uF, base:0603-CAP, symbol base-eagle-import:CAP0603-CAP
- removed C20: 22uF, openmv3:0805, symbol base-eagle-import:CAP0603-CAP
- removed R3: 10K, base:0603-RES, symbol base-eagle-import:RESISTOR0603-RES
- removed R4: 0, base:0603-RES, symbol base-eagle-import:RESISTOR0603-RES
- removed U2: OV7725, openmv3:CSP2-28, symbol base-rescue:OV7725-openmv3-eagle-import
- added C14: 47uF, base:EIA3216, symbol base-eagle-import:CAP_POL1206
- added X3: DF12-36-DS, base:DF12-36-DS, symbol base-eagle-import:DF12-36-DS
- R3: renamed from RN4B1; footprint openmv3:EXBV4V -> base:0603-RES
- R4: renamed from RN4A1; footprint openmv3:EXBV4V -> base:0603-RES
Connections:
- net labels added: RSVD1, RSVD2, RSVD3, RSVD4, RSVD5, RSVD6
- wire segments 313 -> 310
Other:
- moved on the sheet: R3, R4
